File: BugBoard/keypad.kicad_pcb (KiCad board)
At the start: 4 copper layers, 24 x 33 mm, 17 parts, among them J1 USB_B_Micro, J4 Conn_01x06_Pin, U1 PY32F003F18P6TU, U3 XC6206P332MR, U4 NRF24L01_SMD, U5 CH330N

Commit message: PCB update
Parts:
- moved C3 22.8 mm to (144.7, 98.5)
- moved C4 22.8 mm to (144.6, 101.2)
- moved R1 22.8 mm to (143.0, 101.2)
- moved U3 22.8 mm to (147.3, 101.2)
- moved C1 3.73 mm to (155.9, 103.0), turned to 180 degrees
- moved U1 2.42 mm to (154.1, 98.1)
- moved BOOT 0.40 mm to (155.8, 108.8)
Routing:
- net /TX: track 0.00 -> 15.8 mm, vias 0 -> 2
- net GND: track 0.00 -> 12.1 mm, vias 0 -> 1
- net /VBUS: track 0.00 -> 11.7 mm, vias 0 -> 2
- net /USB_D+: track 0.00 -> 9.44 mm
- net /USB_D-: track 0.00 -> 7.81 mm
- net Net-(U5-V3): track 0.00 -> 1.84 mm
- added copper zone on In2.Cu, net +3V3
- added copper zone on In1.Cu, net GND
