File: keypad/Version 3/keypad.kicad_pcb (KiCad board)
At the start: 4 copper layers, 39.9 x 39.9 mm, 34 parts, among them J1 USB_B_Micro, J2 Ext-Batt, J3 IO-Con, J4 Conn_01x06_Pin, J5 IO-Con, SW1 Ident, U1 PY32F003F18P6TU, U2 MAX1555, U3 XC6206P332MR, U4 NRF24L01_SMD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

Commit message: Finished code. Added bug board
Parts:
- moved C7 1.05 mm to (131.2, 82.2)
- moved U5 0.36 mm to (130.9, 86.7)
- moved C5 0.30 mm to (132.5, 94.6)
- moved C6 0.29 mm to (132.0, 91.3)
Routing:
- net Net-(U5-V3): track 8.46 -> 9.91 mm
- net +3V3: track 29.2 -> 29.3 mm, vias 7 -> 6
Other:
- board text added: "Little Monster V1.1"
- board text removed: "Little Monster V1.0"
