File: keypad/Version 4/electronics/keypad.kicad_sch (KiCad schematic)
At the start: 34 parts, among them J1 USB_B_Micro, J2 Ext-Batt, J3 IO-Con, J4 Conn_01x06_Pin, J5 IO-Con, SW1 Ident, U1 PY32F003F18P6TU, U2 TP4054, U3 XC6206P332MR, U4 NRF24L01_SMD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

Commit message: Flash code added and littlefs
Parts:
- J5: now not fitted
- U6: footprint Package_SO:SOIC-8_3.9x4.9mm_P1.27mm -> Package_SO:SOIC-8W_5.3x5.3mm_P1.27mm
Changed lines of the file:
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@@
 			)
 		)
-		(property "Footprint" "Package_SO:SOIC-8_3.9x4.9mm_P1.27mm"
+		(property "Footprint" "Package_SO:SOIC-8W_5.3x5.3mm_P1.27mm"
 			(at 195.58 121.92 0)
 			(effects
@@
 		(exclude_from_sim no)
 		(in_bom yes)
-		(on_board yes)
-		(dnp no)
+		(on_board no)
+		(dnp yes)
 		(fields_autoplaced yes)
 		(property "Reference" "J5"

Commit message: Added basic interpreter (untested)  now adding forth
Parts:
- added R6, R7: 100k, Resistor_SMD:R_0603_1608Metric_Pad0.98x0.95mm_HandSolder, symbol Device:R
Connections:
- net +3V3: now also R6.1, R7.1
- net SWC: now also R7.2
- net SWD: now also R6.2
